File: astable-oscillator.simulation/astable-oscillator.simulation.kicad_sch (KiCad schematic)
At the start: 9 parts, among them Q101 NPN, Q102 NPN

Commit message: Update values for simulation
* Update values for simulation in KiCad.
* Simulation does not converge so we will keep it like this until we
  find a way to fix this.
* Create simulation in LTSpice with the same schematic. This simulation
  gives expected results. It will be kept for comparison with KiCad
  simulation results.
Parts:
- C1: renamed from C101; value 1n -> 1u
- C2: renamed from C102; value 1n -> 1u
- R1: renamed from R104; value 220 -> 100
- R2: renamed from R103; value 220 -> 100k
- R3: renamed from R101; value 220 -> 100k
- R4: renamed from R102; value 220 -> 100
- renumbered Q101 to Q1, Q102 to Q2
Connections:
- net V_{R3-C2-bQ1}: now reaches C2.1, Q1.2 (B), R3.2
- net V_{R1-C1-cQ1}: now reaches C1.1, Q1.1 (C), R1.2
- net V_{BASE} renamed V_{R2-C1-bQ2}
- net V_{COL} renamed V_{R4-C2-cQ2}
Changed lines of the file:
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@@
 		)
 	)
-	(label "V_{COL}"
+	(label "V_{R1-C1-cQ1}"
+		(at 101.6 88.9 180)
+		(effects
+			(font
+				(size 1.25 1.25)
+			)
+			(justify right bottom)
+		)
+	)
+	(label "V_{R4-C2-cQ2}"
 		(at 177.8 88.9 0)
 		(effects
 			(font
-				(size 1.27 1.27)
+				(size 1.25 1.25)
 			)
 			(justify left bottom)
 		)
 	)
-	(label "V_{BASE}"
-		(at 144.78 101.6 0)
+	(label "V_{R2-C1-bQ2}"
+		(at 167.64 101.6 180)
 		(effects
 			(font
-				(size 1.27 1.27)
+				(size 1.25 1.25)
+			)
+			(justify right bottom)
+		)
+	)
+	(label "V_{R3-C2-bQ1}"
+		(at 111.76 101.6 0)
+		(effects
+			(font
+				(size 1.25 1.25)
 			)
 			(justify left bottom)
@@
 		(dnp no)
 		(fields_autoplaced yes)
-		(property "Reference" "R102"
+		(property "Reference" "R4"
 			(at 180.34 78.7399 0)
 			(effects
@@
 			)
 		)
-		(property "Value" "220"
-			(at 180.34 81.2799 0)
-			(effects
-				(font
-					(size 1.27 1.27)
+		(property "Value" "100"
+			(at 180.34 81.28 0)
+			(effects
+				(font
+					(size 1.25 1.25)
 				)
 				(justify left)
@@
 			(project "astable-oscillator.simulation"
 				(path "/f9b52f71-4cc5-45e8-8f08-bf04eea78f5e"
-					(reference "R102")
+					(reference "R4")
 					(unit 1)
 				)
@@
 		(dnp no)
 		(fields_autoplaced yes)
-		(property "Reference" "C102"
+		(property "Reference" "C2"
 			(at 166.37 81.28 90)
 			(effects
@@
 			)
 		)
-		(property "Value" "1n"
+		(property "Value" "1u"
 			(at 166.37 83.82 90)
 			(effects
@@
 			(project "astable-oscillator.simulation"
 				(path "/f9b52f71-4cc5-45e8-8f08-bf04eea78f5e"
-					(reference "C102")
+					(reference "C2")
 					(unit 1)
 				)
@@
 		(on_board yes)
 		(dnp no)
-		(property "Reference" "Q101"
+		(property "Reference" "Q1"
 			(at 98.298 100.3299 0)
 			(effects
@@
 			(project ""
 				(path "/f9b52f71-4cc5-45e8-8f08-bf04eea78f5e"
-					(reference "Q101")
+					(reference "Q1")
 					(unit 1)
 				)
@@
 		(dnp no)
 		(fields_autoplaced yes)
-		(property "Reference" "C101"
+		(property "Reference" "C1"
 			(at 113.03 81.28 90)
 			(effects
@@
 			)
 		)
-		(property "Value" "1n"
+		(property "Value" "1u"
 			(at 113.03 83.82 90)
 			(effects
@@
 			(project ""
 				(path "/f9b52f71-4cc5-45e8-8f08-bf04eea78f5e"
-					(reference "C101")
+					(reference "C1")
 					(unit 1)
 				)
@@
 		(dnp no)
 		(fields_autoplaced yes)
-		(property "Reference" "R103"
+		(property "Reference" "R2"
 			(at 129.54 78.7399 0)
 			(effects
@@
 			)
 		)
-		(property "Value" "220"
-			(at 129.54 81.2799 0)
-			(effects
-				(font
-					(size 1.27 1.27)
+		(property "Value" "100k"
+			(at 129.54 81.28 0)
+			(effects
+				(font
+					(size 1.25 1.25)
 				)
 				(justify left)
@@
 			(project "astable-oscillator.simulation"
 				(path "/f9b52f71-4cc5-45e8-8f08-bf04eea78f5e"
-					(reference "R103")
+					(reference "R2")
 					(unit 1)
 				)
@@
 		(dnp no)
 		(fields_autoplaced yes)
-		(property "Reference" "R104"
+		(property "Reference" "R1"
 			(at 104.14 78.7399 0)
 			(effects
@@
 			)
 		)
-		(property "Value" "220"
-			(at 104.14 81.2799 0)
-			(effects
-				(font
-					(size 1.27 1.27)
+		(property "Value" "100"
+			(at 104.14 81.28 0)
+			(effects
+				(font
+					(size 1.25 1.25)
 				)
 				(justify left)
@@
 			(project "astable-oscillator.simulation"
 				(path "/f9b52f71-4cc5-45e8-8f08-bf04eea78f5e"
-					(reference "R104")
+					(reference "R1")
 					(unit 1)
 				)
@@
 		(dnp no)
 		(fields_autoplaced yes)
-		(property "Reference" "Q102"
-			(at 181.102 100.3299 0)
+		(property "Reference" "Q2"
+			(at 180.34 100.3299 0)
 			(effects
 				(font
@@
 		)
 		(property "Value" "NPN"
-			(at 181.102 102.8699 0)
+			(at 180.34 102.8699 0)
 			(effects
 				(font
@@
 			(project "astable-oscillator.simulation"
 				(path "/f9b52f71-4cc5-45e8-8f08-bf04eea78f5e"
-					(reference "Q102")
+					(reference "Q2")
 					(unit 1)
 				)
@@
 		(dnp no)
 		(fields_autoplaced yes)
-		(property "Reference" "R101"
+		(property "Reference" "R3"
 			(at 154.94 78.7399 0)
 			(effects
@@
 			)
 		)
-		(property "Value" "220"
-			(at 154.94 81.2799 0)
-			(effects
-				(font
-					(size 1.27 1.27)
+		(property "Value" "100k"
+			(at 154.94 81.28 0)
+			(effects
+				(font
+					(size 1.25 1.25)
 				)
 				(justify left)
@@
 			(project ""
 				(path "/f9b52f71-4cc5-45e8-8f08-bf04eea78f5e"
-					(reference "R101")
-					(unit 1)
-				)
+					(reference "R3")
+					(unit 1)
+				)
